File: REALdronePCB/REALdronePCB.kicad_pcb (KiCad board)
At the start: 2 copper layers, 40 x 40 mm, 52 parts, among them IC2 MSPM0G3507SPTR, J1 Conn_01x08_Socket, J2 Conn_01x05, SW5 SW_SPDT, SW6 SW_Push, SW7 SW_RESET, U1 ICM-42688-P, U3 LT1763CS8-3.3_TRPBF, Y2 Crystal_GND24

Commit message: FixedPCB
This is the final version.
Parts:
- moved U1 2.45 mm to (162.8, 82.7)
- moved U3 1.04 mm to (146.0, 86.5)
- moved G*** 0.71 mm to (157.5, 89.0)
- moved REGU-C11 0.71 mm to (151.5, 86.5)
Routing:
- net CH3: track 62.2 -> 71.3 mm
- net GND: track 209.7 -> 201.8 mm
- net SPI1_CS0: track 24.2 -> 30.9 mm
- net C-JST: track 50.2 -> 55.5 mm
- net SPI1_SCK: track 11.7 -> 16.6 mm
- net BOOT: track 34.3 -> 39.2 mm
- net Motor4: track 27.8 -> 31.4 mm
- net CH2: track 29.9 -> 33.4 mm, vias 5 -> 3
- net NRST: track 50.1 -> 52.7 mm, vias 6 -> 5
- net SPI1_PICO: track 15.0 -> 17.7 mm
- net +5V: track 28.8 -> 26.2 mm
- net BUZZER_IO: track 15.3 -> 17.6 mm
- net +3V3: track 150.1 -> 152.3 mm
- net SPI1_POCI: track 12.0 -> 13.7 mm
- net VDD: track 39.5 -> 41.2 mm
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